File: a3921kaitaku.kicad_sch (KiCad schematic)
At the start: 17 parts, among them IC1 A3921KLPTR-T, M1 Motor_DC, Q1 NMOS, Q2 NMOS, Q3 NMOS, Q4 NMOS, U1 Si8640BA-B-IU

Commit message: korosuzo
Parts:
- added C10, C11: 22pF, Capacitor_SMD:C_0603_1608Metric, symbol Device:C
- added C6, C7, C9: 0.1μF, Capacitor_SMD:C_0603_1608Metric, symbol Device:C
- added C8: 22μF, Capacitor_SMD:C_0603_1608Metric, symbol Device:C
- added D2, D3: LED, LED_THT:LED_D3.0mm, symbol Device:LED
- added J1: STlink, symbol Connector:Conn_01x06_Pin
- added J2: CANport, symbol Connector:Conn_01x03_Pin
- added QFF1, QFF2, QRESET: NPN, Package_TO_SOT_SMD:SOT-23, symbol Simulation_SPICE:NPN
- added R10, R11, R12: 10kΩ, Resistor_SMD:R_1206_3216Metric, symbol Device:R
- added R5, R6, R7, R8: 1kΩ, symbol Device:R
- added R9: 1kΩ, Resistor_SMD:R_1206_3216Metric, symbol Device:R
- added U2: STM32F303K8Tx, Package_QFP:LQFP-32_7x7mm_P0.8mm, symbol MCU_ST_STM32F3:STM32F303K8Tx
- added XT1, XT2: ~, Library:Amass_XT60PW-M, symbol XT60:XT60
- added Y1: Crystal, symbol Device:Crystal
- R2: footprint (none) -> Resistor_SMD:R_1206_3216Metric
- renumbered Q1 to Q1H, Q2 to Q1L, Q3 to Q2H, Q4 to Q2L
Connections:
- net -24V is gone; now on net +24V: U1.16 (VDD2)
- net +24V: now also C7.1, XT1.2
- net GND: now also C6.2, C7.2, C8.2, QFF1.3 (E), QFF2.3 (E), QRESET.3 (E), R10.2, XT1.1
- net PHASE: now also U1.11 (B4); no longer U1.12 (B3)
- net SR: now also U1.12 (B3); no longer U1.11 (B4)
- net V5: now also R5.1, R6.1, R9.1
- net +3.3V: now reaches U1.1 (VDD1)
- net +3.3V: now also J1.1 (Pin_1), R11.1, U2.1 (VDD), U2.17 (VDD), U2.5 (VDDA), XT2.2
- net GND1: now reaches U1.2 (GND1), U1.8 (GND1)
- net GND1: now also C10.2, C11.2, C9.2, J1.3 (Pin_3), J2.3 (Pin_3), R12.2, U2.16 (VSS), U2.32 (VSS), XT2.1
- net RESET: now reaches IC1.24 (RESET)
- net RESET: now also QRESET.1 (C)
- net FF1: now reaches IC1.25 (FF1)
- net FF1: now also R8.1
- net FF2: now reaches IC1.26 (FF2)
- net FF2: now also R7.2
- net VDSTH: now reaches IC1.28 (VDSTH)
- net VDSTH: now also R10.1, R9.2
- net VREG: now reaches IC1.8 (VREG)
- net VREG: now also C6.1, C8.1
- new net: D3.1 (K), QFF2.1 (C)
- new net: D3.2 (A), R6.2
- new net: QFF2.2 (B), R7.1
- new net: D2.1 (K), QFF1.1 (C)
- new net: D2.2 (A), R5.2
- new net: QFF1.2 (B), R8.2
- new net BOOT0: R12.1, U2.31 (BOOT0)
- new net NRST: C9.1, J1.5 (Pin_5), R11.2, U2.4 (NRST)
- new net PA13: J1.4 (Pin_4), U2.23 (PA13)
- new net PA14: J1.2 (Pin_2), U2.24 (PA14)
- new net PB3: J1.6 (Pin_6), U2.26 (PB3)
- new net PB4: U2.27 (PB4)
- new net PF0: C10.1, U2.2 (PF0), Y1.1
- new net PF1: C11.1, U2.3 (PF1), Y1.2
- new net RX: J2.2 (Pin_2), U2.20 (PA10)
- new net TX: J2.1 (Pin_1), U2.19 (PA9)
- no-connect marks 3 -> 4
Other:
- note added: "IC"
- note added: "アイソレータ"
- note added: "パスコン"
- note added: "モータ駆動部"
- note added: "故障確認LED"
- note added: "電源"
- moved on the sheet: C2, C3, C4, C5, IC1, M1, Q1H, Q1L, Q2H, Q2L, R1, R2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

Commit message: unti
Parts:
- removed Q1H, Q1L, Q2H, Q2L: NMOS, symbol Simulation_SPICE:NMOS
- added C12, C13, C14: 0.1μF, Capacitor_SMD:C_0603_1608Metric, symbol Device:C
- added D4: LED, LED_THT:LED_D3.0mm, symbol Device:LED
- added Q1: Q1H, Package_TO_SOT_SMD:TO-252-2, symbol Transistor_FET:QM6006D
- added Q2: Q2H, Package_TO_SOT_SMD:TO-252-2, symbol Transistor_FET:QM6006D
- added Q3: Q1L, Package_TO_SOT_SMD:TO-252-2, symbol Transistor_FET:QM6006D
- added Q4: Q2L, Package_TO_SOT_SMD:TO-252-2, symbol Transistor_FET:QM6006D
- added R13, R14: 1kΩ, Resistor_SMD:R_1206_3216Metric, symbol Device:R
- added R15, R16, R17, R18: 22Ω, Resistor_SMD:R_1206_3216Metric, symbol Device:R
- added R19, R20: 47kΩ, Resistor_SMD:R_1206_3216Metric, symbol Device:R
- added R21: 330kΩ, Resistor_SMD:R_1206_3216Metric, symbol Device:R
- added U3: LF33_TO252, Package_TO_SOT_SMD:TO-252-2, symbol Regulator_Linear:LF33_TO252
- IC1: footprint a3921:A3944KLPTRT -> Library:A3944KLPTRT
- J1: footprint (none) -> Connector_PinHeader_2.54mm:PinHeader_1x06_P2.54mm_Vertical
- J2: footprint (none) -> Connector_PinHeader_2.54mm:PinHeader_1x03_P2.54mm_Vertical
- M1: footprint Amass_XT60PW-M_footprints:Amass_XT60PW-M -> Library:Amass_XT60PW-M
- R1: value 3kΩ -> 9.1kΩ
- R2: value R -> 47kΩ
- R4: value R -> 47kΩ; footprint (none) -> Resistor_SMD:R_1206_3216Metric
- R5, R6: footprint (none) -> Resistor_SMD:R_1206_3216Metric
- R7, R8: value 1kΩ -> 10kΩ; footprint (none) -> Resistor_SMD:R_1206_3216Metric
- Y1: value Crystal -> 48MHz; footprint (none) -> Crystal:Crystal_HC49-U_Vertical
- renumbered QRESET to QRESET1
Connections:
- net +24V: now also Q1.2 (D), Q2.2 (D)
- net +3.3V: now also C12.1, C13.1, C14.1, U3.3 (VO); no longer XT2.2
- net FF1: now also R14.2
- net FF2: now also R13.2
- net GHA: now also R16.1; no longer R4.1
- net GHB: now also R15.2; no longer R2.1
- net GLA: now also R18.1
- net GLB: now also R17.2
- net GND: now also Q3.3 (S), Q4.3 (S), R19.2, R20.2
- net GND1: now also C12.2, C13.2, C14.2, D4.1 (K), U3.2 (GND)
- net SA: now also Q1.3 (S), Q3.2 (D); no longer C4.2
- net SB: now also C4.2, Q2.3 (S), Q4.2 (D)
- net V5: now also R13.1, R14.1
- net PA6: now reaches QRESET1.2 (B)
- net PA6: now also U2.22 (PA12)
- net PA4: now reaches U2.10 (PA4)
- net PA4: now also U1.5 (A3)
- net PA5: now reaches U2.11 (PA5)
- net PA5: now also U1.6 (A4)
- net PA8: now reaches U2.18 (PA8)
- net PA8: now also U1.3 (A1)
- net PA11: now reaches U2.21 (PA11)
- net PA11: now also U1.4 (A2)
- net PB7: now reaches U2.30 (PB7)
- net PB7: now also R21.2
- new net: Q4.1 (G), R17.1, R20.1
- new net: Q3.1 (G), R18.2, R19.1
- new net: Q1.1 (G), R16.2, R4.1
- new net: D4.2 (A), R21.1
- new net: Q2.1 (G), R15.1, R2.1
- new net +12V: U3.1 (VI), XT2.2
Other:
- note added: "コネクタ"
- note added: "マイコン"
- moved on the sheet: C1, C10, C11, D1, D2, D3, IC1, J1, J2, M1, QFF1, QFF2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

Commit message: unchiunchi
Parts:
- removed IC1: A3921KLPTR-T, Library:A3944KLPTRT, symbol A3921KLPTR-T:A3921KLPTR-T
- added C15, C16, C18: 0.1μF, Capacitor_SMD:C_0603_1608Metric, symbol Device:C
- added C17: 4.7μF, Capacitor_SMD:C_0603_1608Metric, symbol Device:C
- added D5, D6, D7, D8, D9: D, Diode_SMD:D_1206_3216Metric, symbol Device:D
- added IC1: A3921KLPTR-T, A3944KLPTRT, symbol A3921:A3921KLPTR-T
- added J3, J4: Conn_01x02_Pin, Connector_PinHeader_2.54mm:PinHeader_1x02_P2.54mm_Horizontal, symbol Connector:Conn_01x02_Pin
- added R22: 300Ω, Resistor_SMD:R_1206_3216Metric, symbol Device:R
- added R23, R24: 60Ω, Resistor_SMD:R_1206_3216Metric, symbol Device:R
- added R25: 100kΩ, Resistor_SMD:R_1206_3216Metric, symbol Device:R
- added SW1: SW_DIP_x02, Button_Switch_THT:SW_DIP_SPSTx02_Slide_9.78x7.26mm_W7.62mm_P2.54mm, symbol Switch:SW_DIP_x02
- added U4: MCP2561-E-SN, Package_DIP:DIP-8_W7.62mm, symbol Interface_CAN_LIN:MCP2561-E-SN
- added U5: LF50_TO252, Package_TO_SOT_SMD:TO-252-2, symbol Regulator_Linear:LF50_TO252
- J2: value CANport -> UARTport
Connections:
- net +12V: now also U5.1 (VI)
- net +24V: now also C16.2, D5.2 (A), D6.1 (K), D7.1 (K), IC1.1 (VDRAIN)
- net +3.3V: now also C15.1
- net CA: now also IC1.9 (CA)
- net CB: now also IC1.6 (CB)
- net CP1: now also IC1.16 (CP1)
- net CP2: now also IC1.15 (CP2)
- net FF1: now also IC1.25 (FF1)
- net FF2: now also IC1.26 (FF2)
- net GHA: now also IC1.10 (GHA)
- net GHB: now also IC1.5 (GHB)
- net GLA: now also IC1.12 (GLA)
- net GLB: now also IC1.3 (GLB)
- net GND: now also C16.1, D8.2 (A), D9.2 (A), IC1.17 (GND), IC1.2 (LSS)
- net GND1: now also C15.2, C17.2, C18.2, R25.1, U4.2 (VSS), U5.2 (GND)
- net PA5: now also U1.3 (A1); no longer U1.6 (A4)
- net PA6: now also U2.12 (PA6); no longer U2.22 (PA12)
- net PA8: now also U1.6 (A4); no longer U1.3 (A1)
- net PHASE: now also U1.14 (B1), IC1.19 (PHASE); no longer U1.11 (B4)
- net PWMH: now also U1.11 (B4), IC1.23 (PWMH); no longer U1.14 (B1)
- net PWML: now also U1.12 (B3), IC1.22 (PWML); no longer U1.13 (B2)
- net RDEAD: now also IC1.27 (RDEAD)
- net RESET: now also IC1.24 (RESET)
- net RX: now also U2.10 (PA4); no longer U2.20 (PA10)
- net SA: now also D6.2 (A), D8.1 (K), IC1.11 (SA)
- net SB: now also D7.2 (A), D9.1 (K), IC1.4 (SB)
- net SR: now also U1.13 (B2), IC1.21 (SR); no longer U1.12 (B3)
- net TX: now also U2.9 (PA3); no longer U2.19 (PA9)
- net V5: now also IC1.20 (V5)
- net VDSTH: now also IC1.28 (VDSTH)
- net VREG: now also IC1.8 (VREG)
- net PA7: now reaches U2.13 (PA7)
- net PA7: now also U1.4 (A2)
- net PA11 renamed CAN_RX
- net CAN_RX: now also U4.4 (RXD); no longer U1.4 (A2)
- net PA4 renamed PA9
- net PA9: now also U2.19 (PA9); no longer U2.10 (PA4)
- new net: D5.1 (K), IC1.13 (VBB)
- new net: R23.1, SW1.3
- new net: C17.1, R22.2, R23.2, R24.2
- new net: R24.1, SW1.4
- new net: R25.2, U4.8 (STBY)
- new net +5V: C18.1, U4.3 (VDD), U5.3 (VO)
- new net CANH: J3.2 (Pin_2), J4.2 (Pin_2), SW1.2, U4.6 (CANL)
- new net CANL: J3.1 (Pin_1), J4.1 (Pin_1), SW1.1, U4.7 (CANH)
- new net CAN_TX: U2.22 (PA12), U4.1 (TXD)
- new net SPLIT: R22.1, U4.5 (SPLIT)
- no-connect marks 4 -> 5
Other:
- note added: "CANトランシーバ"
- moved on the sheet: D2, D3, J1, J2, QFF1, QFF2, R13, R14, R5, R6, R7, R8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
